Commit message: Add files via upload

File: models/kinova/j2s7s300_withBase.xacro (robot description, xacro)
@@ -14,5 +14,4 @@
     xmlns:physics="http://playerstage.sourceforge.net/gazebo/xmlschema/#physics"
 	xmlns:xacro="http://ros.org/wiki/xacro" name="j2s7s300">
-  <xacro:include filename="$(find robot_grasp)/models/table/table_simple.xacro"/>
   <xacro:include filename="$(find robot_grasp)/models/table/table.xacro"/>
   <xacro:include filename="$(find kinova_description)/urdf/j2s7s300.xacro"/>
@@ -21,17 +20,4 @@
     <material>Gazebo/FlatBlack</material>
   </gazebo>
-       <link name="world" />
-	<joint name="j0" type="fixed">
-		<origin xyz="0 0 0.273" rpy="0 0 0" />
-		<parent link="world" />
-		<child link="table_base" />
-		<axis xyz="0 0 0" />
-	</joint>
-	<joint name="j02" type="fixed">
-		<origin xyz="0 0.85 0.273" rpy="0 0 0" />
-		<parent link="world" />
-		<child link="table_base2" />
-		<axis xyz="0 0 0" />
-	</joint>
   <link name="arm_stand">
     <inertial>
@@ -58,5 +44,5 @@
   <joint name="j2b" type="fixed">
     <origin rpy="-1.57079632679 -3.14159265358979 0" xyz="0 -0.035 0"/>
-    <parent link="tabletop_corner2"/>
+    <parent link="tabletop_corner"/>
     <child link="arm_stand"/>
     <axis xyz="0 0 0"/>
@@ -80,5 +66,5 @@
     <child link="root" />
     <parent link="arm_stand" />
-    <origin xyz="0 0.08 0" rpy="-1.57079632679 1.57079632679 0" />
+    <origin xyz="0 0.08 0" rpy="-1.57079632679 0.05 0" />
   </joint>
   <property name="robot_root" value="root" />

File: models/table/table.xacro (robot description, xacro)
@@ -1,4 +1,3 @@
-<?xml version="1.0"?>
-<!-- j2s7s300 refers to jaco v2 7DOF spherical 3fingers -->
+<?xml version="1.0" encoding="UTF-8"?>
 <root xmlns:xacro="http://ros.org/wiki/xacro">
 	<xacro:include filename="$(find robot_grasp)/models/table/table_properties.xacro" />
@@ -84,4 +83,11 @@
 	</link>
 <!-- Added   -->
+       <link name="world" />
+	<joint name="j0" type="fixed">
+		<origin xyz="0 0 0.273" rpy="0 0 0" />
+		<parent link="world" />
+		<child link="table_base" />
+		<axis xyz="0 0 0" />
+	</joint>
 	<joint name="j1" type="fixed">
 		<origin xyz="0.0185115091791201 -0.175991980646074 0.397575968372377" rpy="1.5707963267949 0 0" />
@@ -106,14 +112,8 @@
         <!-- Grasp Objects -->
 	<gazebo reference="basket">
-          <mu1>100.0</mu1>
-          <mu2>100.0</mu2>
-          <minDepth>0.01</minDepth>
-          <material>Gazebo/Green</material>
+		<material>Gazebo/Green</material>
 	</gazebo>
 	<gazebo reference="basket2">
-          <mu1>100.0</mu1>
-          <mu2>100.0</mu2>
-          <minDepth>0.01</minDepth>
-          <material>Gazebo/Blue</material>
+		<material>Gazebo/Blue</material>
 	</gazebo>
 	<gazebo reference="kinect_support">
@@ -129,11 +129,11 @@
 			<origin xyz="0 0 -0.1" rpy="0 0 0" />
 			<geometry>
-                                <mesh scale="0.0013 0.0013 0.0013" filename="$(find robot_grasp)/models/grasp_object/basket.dae" />
-			</geometry>
-		</visual>
-		<collision>
-			<origin xyz="0 0 -0.1" rpy="0 0 0" />
-			<geometry>
-                                <mesh scale="0.0013 0.0013 0.0013" filename="$(find robot_grasp)/models/grasp_object/basket.dae" />
+				<mesh scale="0.001 0.001 0.001" filename="$(find robot_grasp)/models/grasp_object/basket.dae" />
+			</geometry>
+		</visual>
+		<collision>
+			<origin xyz="0 0 -0.1" rpy="0 0 0" />
+			<geometry>
+				<mesh scale="0.001 0.001 0.001" filename="$(find robot_grasp)/models/grasp_object/basket.dae" />
 			</geometry>
 		</collision>
@@ -148,11 +148,11 @@
 			<origin xyz="0 0 -0.1" rpy="0 0 0" />
 			<geometry>
-                                <mesh scale="0.001 0.001 0.001" filename="$(find robot_grasp)/models/grasp_object/basket.dae" />
-			</geometry>
-		</visual>
-		<collision>
-			<origin xyz="0 0 -0.1" rpy="0 0 0" />
-			<geometry>
-                                <mesh scale="0.0008 0.0008 0.0008" filename="$(find robot_grasp)/models/grasp_object/basket.dae" />
+				<mesh scale="0.001 0.001 0.001" filename="$(find robot_grasp)/models/grasp_object/basket.dae" />
+			</geometry>
+		</visual>
+		<collision>
+			<origin xyz="0 0 -0.1" rpy="0 0 0" />
+			<geometry>
+				<mesh scale="0.001 0.001 0.001" filename="$(find robot_grasp)/models/grasp_object/basket.dae" />
 			</geometry>
 		</collision>
@@ -173,10 +173,10 @@
 			<origin xyz="0 0 0" rpy="0 0 0" />
 			<geometry>
-				<mesh scale="0.001 0.001 0.001" filename="$(find robot_grasp)/models/table/meshes/kinect_support.dae" />
+				<mesh scale="0.001 0.001 0.001" filename="$(find robot_grasp)/models/grasp_object/meshes/kinect_support.dae" />
 			</geometry>
 		</collision>
 	</link>
 	<joint name="table_basket" type="fixed">
-                <origin xyz="0.25 0.065 0.1" rpy="0 0 0" />  <!-- relative to world coordinator: y z x 0.25 0.06 0.1-->
+		<origin xyz="0.25 0.06 0.15" rpy="0 0 0" />  <!-- relative to world coordinator: y z x -->
 		<parent link="table_top" />
 		<child link="basket" />
@@ -184,5 +184,5 @@
 	</joint>
 	<joint name="table_basket2" type="fixed">
-                <origin xyz="-0.25 0.06 0.1" rpy="0 0 0" />
+		<origin xyz="-0.2 0.06 0.15" rpy="0 0 0" />
 		<parent link="table_top" />
 		<child link="basket2" />
@@ -190,96 +190,9 @@
 	</joint>
 	<joint name="table_kinect_support" type="fixed">
-                <origin xyz="0.1 0.19 0.25" rpy="0 -1.5707963267949 0" />  <!-- relative to world coordinator: x z -y -->
+		<origin xyz="0.1 0.19 0.3" rpy="0 -1.5707963267949 0" />  <!-- relative to world coordinator: x z -y -->
 		<parent link="table_top" />
 		<child link="kinect_support" />
 		<axis xyz="0 0 0" />
 	</joint>
-    <link name="camera_link">
-            <collision>
-              <origin xyz="-0.016 0 0" rpy="0 0 0"/>
-              <geometry>
-                <box size="0.036 0.18 0.04"/>
-              </geometry>
-            </collision>
-            <visual>
-              <origin xyz="0 0 0" rpy="0 0 0"/>
-              <geometry>
-                <mesh filename="package://robot_grasp/models/kinect/meshes/kinect.dae"/>
-              </geometry>
-            </visual>
-            <inertial>
-              <mass value="1.0" />
-              <origin xyz="0 0 0" rpy="0 0 0"/>
-              <inertia ixx="5.8083e-4" ixy="0" ixz="0" iyy="3.0833e-5" iyz="0" izz="5.9083e-4" />
-            </inertial>
-         </link>
-        <joint name="camera_joint" type="fixed">
-            <origin xyz="-0.25 0.48 0" rpy="1.5707963267949 0 -1.5707963267949" /><!--"-0.278 0.41 0" -->
-            <parent link="kinect_support" />
-            <child link="camera_link" />
-            <axis xyz="0 1 0"/>
-        </joint>
-        <link name="camera_rgb_frame" />
-          <joint name="camera_rgb_joint" type="fixed">
-            <origin rpy="0 0 0" xyz="0 0.022 0" />
-            <parent link="camera_link" />
-            <child link="camera_rgb_frame" />
-          </joint>
-          <link name="camera_rgb_optical_frame" />
-          <joint name="camera_rgb_optical_joint" type="fixed">
-            <origin rpy="-1.57079632679 0 -1.57079632679" xyz="0 0 0" />
-            <parent link="camera_rgb_frame" />
-            <child link="camera_rgb_optical_frame" />
-          </joint>
-          <link name="camera_depth_frame" />
-          <joint name="camera_depth_joint" type="fixed">
-            <origin rpy="0 0 0" xyz="0 0.049 0" />
-            <parent link="camera_link" />
-            <child link="camera_depth_frame" />
-          </joint>
-          <link name="camera_depth_optical_frame" />
-          <joint name="camera_depth_optical_joint" type="fixed">
-            <origin rpy="-1.57079632679 0 -1.57079632679" xyz="0 0 0" />
-            <parent link="camera_depth_frame" />
-            <child link="camera_depth_optical_frame" />
-          </joint>
-        <gazebo reference="camera_rgb_frame">
-            <sensor type="depth" name="camera">
-              <always_on>true</always_on>
-              <visualize>false</visualize>
-              <update_rate>15.0</update_rate>
-              <camera name="front">
-                <horizontal_fov>1.047197</horizontal_fov>
-                <image>
-                  <format>B8G8R8</format>
-                  <width>1920</width>
-                  <height>1080</height>
-                </image>
-                <clip>
-                  <near>0.01</near>
-                  <far>9</far>
-                </clip>
-              </camera>
-              <plugin name="camera_controller" filename="libgazebo_ros_openni_kinect.so">
-                <baseline>0.1</baseline>
-                <alwaysOn>true</alwaysOn>
-                <updateRate>15.0</updateRate>
-                <cameraName>camera</cameraName>
-                <imageTopicName>/camera/rgb/image_raw</imageTopicName>
-                <cameraInfoTopicName>/camera/rgb/camera_info</cameraInfoTopicName>
-                <depthImageTopicName>/camera/depth_registered/image_raw</depthImageTopicName>
-                <depthImageCameraInfoTopicName>/camera/depth_registered/camera_info</depthImageCameraInfoTopicName>
-                <pointCloudTopicName>/camera/depth_registered/points</pointCloudTopicName>
-                <frameName>camera_rgb_optical_frame</frameName>
-                <pointCloudCutoff>0.35</pointCloudCutoff>
-                <pointCloudCutoffMax>4.5</pointCloudCutoffMax>
-                <CxPrime>0</CxPrime>
-                <Cx>900</Cx>
-                <Cy>540</Cy>
-                <focalLength>1.0</focalLength>
-                <hackBaseline>0</hackBaseline>
-              </plugin>
-            </sensor>
-          </gazebo>
  <!--       <gazebo reference="cubic">
 	        <material>Gazebo/Yellow</material>

File: models/table/table_properties.xacro (robot description, xacro)
@@ -6,13 +6,3 @@
   <xacro:property name="rim_height" value="0.015"/>
   <xacro:property name="rim_thickness" value="0.005"/>
-  <!--Define constants-->
-    <xacro:property name="PI" value="3.14159"/>
-    <xacro:property name="mass1" value="10" />
-    <xacro:property name="mass2" value="1" />
-    <xacro:property name="width1" value="0.1" />
-    <xacro:property name="width2" value="0.1" />
-    <xacro:property name="length0" value="0.1" />
-    <xacro:property name="length1" value="1.5" />
-    <xacro:property name="length2" value="0.1" />
-    <xacro:property name="mass_camera" value="0.2" />
 </root>

Commit message: Add files via upload

File: models/kinova/j2s7s300_withBase.xacro (robot description, xacro)
@@ -80,5 +80,5 @@
     <child link="root" />
     <parent link="arm_stand" />
-    <origin xyz="0 0.08 0" rpy="-1.57079632679 1.57079632679 0" />
+    <origin xyz="0 0.08 0" rpy="-1.57079632679 0.05 0" />
   </joint>
   <property name="robot_root" value="root" />

File: models/table/table.xacro (robot description, xacro)
@@ -106,14 +106,8 @@
         <!-- Grasp Objects -->
 	<gazebo reference="basket">
-          <mu1>100.0</mu1>
-          <mu2>100.0</mu2>
-          <minDepth>0.01</minDepth>
-          <material>Gazebo/Green</material>
+		<material>Gazebo/Green</material>
 	</gazebo>
 	<gazebo reference="basket2">
-          <mu1>100.0</mu1>
-          <mu2>100.0</mu2>
-          <minDepth>0.01</minDepth>
-          <material>Gazebo/Blue</material>
+		<material>Gazebo/Blue</material>
 	</gazebo>
 	<gazebo reference="kinect_support">
@@ -129,11 +123,11 @@
 			<origin xyz="0 0 -0.1" rpy="0 0 0" />
 			<geometry>
-                                <mesh scale="0.0013 0.0013 0.0013" filename="$(find robot_grasp)/models/grasp_object/basket.dae" />
-			</geometry>
-		</visual>
-		<collision>
-			<origin xyz="0 0 -0.1" rpy="0 0 0" />
-			<geometry>
-                                <mesh scale="0.0013 0.0013 0.0013" filename="$(find robot_grasp)/models/grasp_object/basket.dae" />
+				<mesh scale="0.0012 0.0012 0.0012" filename="$(find robot_grasp)/models/grasp_object/basket.dae" />
+			</geometry>
+		</visual>
+		<collision>
+			<origin xyz="0 0 -0.1" rpy="0 0 0" />
+			<geometry>
+				<mesh scale="0.0012 0.0012 0.0012" filename="$(find robot_grasp)/models/grasp_object/basket.dae" />
 			</geometry>
 		</collision>
@@ -148,11 +142,11 @@
 			<origin xyz="0 0 -0.1" rpy="0 0 0" />
 			<geometry>
-                                <mesh scale="0.001 0.001 0.001" filename="$(find robot_grasp)/models/grasp_object/basket.dae" />
-			</geometry>
-		</visual>
-		<collision>
-			<origin xyz="0 0 -0.1" rpy="0 0 0" />
-			<geometry>
-                                <mesh scale="0.0008 0.0008 0.0008" filename="$(find robot_grasp)/models/grasp_object/basket.dae" />
+				<mesh scale="0.001 0.001 0.001" filename="$(find robot_grasp)/models/grasp_object/basket.dae" />
+			</geometry>
+		</visual>
+		<collision>
+			<origin xyz="0 0 -0.1" rpy="0 0 0" />
+			<geometry>
+				<mesh scale="0.001 0.001 0.001" filename="$(find robot_grasp)/models/grasp_object/basket.dae" />
 			</geometry>
 		</collision>
@@ -173,10 +167,10 @@
 			<origin xyz="0 0 0" rpy="0 0 0" />
 			<geometry>
-				<mesh scale="0.001 0.001 0.001" filename="$(find robot_grasp)/models/table/meshes/kinect_support.dae" />
+				<mesh scale="0.001 0.001 0.001" filename="$(find robot_grasp)/models/grasp_object/meshes/kinect_support.dae" />
 			</geometry>
 		</collision>
 	</link>
 	<joint name="table_basket" type="fixed">
-                <origin xyz="0.25 0.065 0.1" rpy="0 0 0" />  <!-- relative to world coordinator: y z x 0.25 0.06 0.1-->
+		<origin xyz="0.25 0.06 0.15" rpy="0 0 0" />  <!-- relative to world coordinator: y z x -->
 		<parent link="table_top" />
 		<child link="basket" />
@@ -184,5 +178,5 @@
 	</joint>
 	<joint name="table_basket2" type="fixed">
-                <origin xyz="-0.25 0.06 0.1" rpy="0 0 0" />
+		<origin xyz="-0.2 0.06 0.15" rpy="0 0 0" />
 		<parent link="table_top" />
 		<child link="basket2" />
@@ -190,96 +184,9 @@
 	</joint>
 	<joint name="table_kinect_support" type="fixed">
-                <origin xyz="0.1 0.19 0.25" rpy="0 -1.5707963267949 0" />  <!-- relative to world coordinator: x z -y -->
+		<origin xyz="0.1 0.19 0.3" rpy="0 -1.5707963267949 0" />  <!-- relative to world coordinator: x z -y -->
 		<parent link="table_top" />
 		<child link="kinect_support" />
 		<axis xyz="0 0 0" />
 	</joint>
-    <link name="camera_link">
-            <collision>
-              <origin xyz="-0.016 0 0" rpy="0 0 0"/>
-              <geometry>
-                <box size="0.036 0.18 0.04"/>
-              </geometry>
-            </collision>
-            <visual>
-              <origin xyz="0 0 0" rpy="0 0 0"/>
-              <geometry>
-                <mesh filename="package://robot_grasp/models/kinect/meshes/kinect.dae"/>
-              </geometry>
-            </visual>
-            <inertial>
-              <mass value="1.0" />
-              <origin xyz="0 0 0" rpy="0 0 0"/>
-              <inertia ixx="5.8083e-4" ixy="0" ixz="0" iyy="3.0833e-5" iyz="0" izz="5.9083e-4" />
-            </inertial>
-         </link>
-        <joint name="camera_joint" type="fixed">
-            <origin xyz="-0.25 0.48 0" rpy="1.5707963267949 0 -1.5707963267949" /><!--"-0.278 0.41 0" -->
-            <parent link="kinect_support" />
-            <child link="camera_link" />
-            <axis xyz="0 1 0"/>
-        </joint>
-        <link name="camera_rgb_frame" />
-          <joint name="camera_rgb_joint" type="fixed">
-            <origin rpy="0 0 0" xyz="0 0.022 0" />
-            <parent link="camera_link" />
-            <child link="camera_rgb_frame" />
-          </joint>
-          <link name="camera_rgb_optical_frame" />
-          <joint name="camera_rgb_optical_joint" type="fixed">
-            <origin rpy="-1.57079632679 0 -1.57079632679" xyz="0 0 0" />
-            <parent link="camera_rgb_frame" />
-            <child link="camera_rgb_optical_frame" />
-          </joint>
-          <link name="camera_depth_frame" />
-          <joint name="camera_depth_joint" type="fixed">
-            <origin rpy="0 0 0" xyz="0 0.049 0" />
-            <parent link="camera_link" />
-            <child link="camera_depth_frame" />
-          </joint>
-          <link name="camera_depth_optical_frame" />
-          <joint name="camera_depth_optical_joint" type="fixed">
-            <origin rpy="-1.57079632679 0 -1.57079632679" xyz="0 0 0" />
-            <parent link="camera_depth_frame" />
-            <child link="camera_depth_optical_frame" />
-          </joint>
-        <gazebo reference="camera_rgb_frame">
-            <sensor type="depth" name="camera">
-              <always_on>true</always_on>
-              <visualize>false</visualize>
-              <update_rate>15.0</update_rate>
-              <camera name="front">
-                <horizontal_fov>1.047197</horizontal_fov>
-                <image>
-                  <format>B8G8R8</format>
-                  <width>1920</width>
-                  <height>1080</height>
-                </image>
-                <clip>
-                  <near>0.01</near>
-                  <far>9</far>
-                </clip>
-              </camera>
-              <plugin name="camera_controller" filename="libgazebo_ros_openni_kinect.so">
-                <baseline>0.1</baseline>
-                <alwaysOn>true</alwaysOn>
-                <updateRate>15.0</updateRate>
-                <cameraName>camera</cameraName>
-                <imageTopicName>/camera/rgb/image_raw</imageTopicName>
-                <cameraInfoTopicName>/camera/rgb/camera_info</cameraInfoTopicName>
-                <depthImageTopicName>/camera/depth_registered/image_raw</depthImageTopicName>
-                <depthImageCameraInfoTopicName>/camera/depth_registered/camera_info</depthImageCameraInfoTopicName>
-                <pointCloudTopicName>/camera/depth_registered/points</pointCloudTopicName>
-                <frameName>camera_rgb_optical_frame</frameName>
-                <pointCloudCutoff>0.35</pointCloudCutoff>
-                <pointCloudCutoffMax>4.5</pointCloudCutoffMax>
-                <CxPrime>0</CxPrime>
-                <Cx>900</Cx>
-                <Cy>540</Cy>
-                <focalLength>1.0</focalLength>
-                <hackBaseline>0</hackBaseline>
-              </plugin>
-            </sensor>
-          </gazebo>
  <!--       <gazebo reference="cubic">
 	        <material>Gazebo/Yellow</material>
